Commit message: Created launch file that launches gazebo, world and model, created a ros-gazebo bridge config file

File: description/robot.urdf.xacro (robot description, xacro)
@@ -1,4 +1,5 @@
 <?xml version="1.0"?>
-<robot xmlns:xacro="http://www.ros.org/wiki/xacro" name="robot">
-    <xacro:include filename="robot_core.xacro" />
+<robot xmlns:xacro="http://www.ros.org/wiki/xacro" name="differential_drive_robot">
+    <xacro:include filename="robot_core.xacro"/>
+    <xacro:include filename="gazebo_control.xacro"/>
 </robot>

File: description/robot_core.xacro (robot description, xacro)
@@ -46,4 +46,5 @@
         <child link="left_wheel"/>
         <origin xyz="0 0.175 0" rpy="-${pi/2} 0 0" />
+        <limit effort="50000" velocity="10"/>
         <axis xyz="0 0 1"/>
     </joint>
@@ -69,4 +70,5 @@
         <child link="right_wheel"/>
         <origin xyz="0 -0.175 0" rpy="${pi/2} 0 0" />
+        <limit effort="50000" velocity="10"/>
         <axis xyz="0 0 -1"/>
     </joint>
