Commit message: Add simulation, ros2_control, sensors, bridge and test program
Restores the local work on top of origin/main: launch file, ros2_control and controller parameters, lidar and camera, bridge reduced to clock, scan and camera, package.xml and CMakeLists updates, test world, src/test.cpp, README and .gitignore.

File: description/gazebo_control.xacro (robot description, xacro)
@@ -14,4 +14,7 @@
         <mu1 value="0.001"/>
         <mu2 value="0.001"/>
+    </gazebo>
+    <gazebo reference="camera_link">
+        <material>Gazebo/Red</material>
     </gazebo>
     <gazebo>

File: description/robot.urdf.xacro (robot description, xacro)
@@ -2,5 +2,8 @@
 <robot xmlns:xacro="http://www.ros.org/wiki/xacro" name="differential_drive_robot">
     <xacro:include filename="robot_core.xacro"/>
-    <xacro:include filename="gazebo_control.xacro"/>
+    <!-- <xacro:include filename="gazebo_control.xacro"/> -->
+    <xacro:include filename="ros2_control.xacro"/>
     <xacro:include filename="lidar.xacro"/>
+    <xacro:include filename="camera.xacro"/>
+    <!-- <xacro:include filename="depth_camera.xacro"/> -->
 </robot>

File: description/robot_core.xacro (robot description, xacro)
@@ -13,4 +13,7 @@
     <material name="black">
         <color rgba="0 0 0 1"/>
+    </material>
+    <material name="red">
+        <color rgba="1 0 0 1"/>
     </material>
     <!-- BASE LINK -->
@@ -111,3 +114,9 @@
         </xacro:inertial_sphere>
     </link>
+    <!-- Include for ros2_control.xacro -->
+    <gazebo reference="caster_wheel">
+        <material>Gazebo/Black</material>
+        <mu1 value="0.001"/>
+        <mu2 value="0.001"/>
+    </gazebo>
 </robot>
